Commit message: Fixed orientation of the base_link of the robot for navigation stack.

File: trunk/hydro/robone/robone_description/urdf/main.xacro (robot description, xacro)
@@ -38,8 +38,8 @@
   </link>
   <xacro:motor_wheel suffix="right" width="${wheel_width}" radius="${wheel_radius}"
-       x_shift="${base_radius/2}" y_shift="${-base_radius/2}" z_shift="${-base_height/2}"/>
+       x_shift="${-base_radius/2}" y_shift="${-base_radius/2}" z_shift="${-base_height/2}"/>
   <xacro:motor_wheel suffix="left" width="${wheel_width}" radius="${wheel_radius}"
-       x_shift="${-base_radius/2}" y_shift="${-base_radius/2}" z_shift="${-base_height/2}"/>
+       x_shift="${-base_radius/2}" y_shift="${base_radius/2}" z_shift="${-base_height/2}"/>
   <xacro:simple_wheel suffix="forward" width="${wheel_width}" radius="${wheel_radius}"
-       y_shift="${base_radius/2}" z_shift="${-base_height/2}"/>
+       x_shift="${base_radius/2}" z_shift="${-base_height/2}"/>
 </robot>

File: trunk/hydro/robone/robone_description/urdf/wheel.xacro (robot description, xacro)
@@ -31,5 +31,5 @@
       <parent link="${suffix}_wheel_holder"/>
       <child link="${suffix}_wheel"/>
-      <origin xyz="${wheel_holder_width/2 + width/2} 0 ${-radius/2 - wheel_holder_width/2}" rpy="0 ${-pi/2} 0" />
+      <origin xyz="0 ${wheel_holder_width/2 + width/2} ${-radius/2 - wheel_holder_width/2}" rpy="0 ${-pi/2} ${-pi/2}" />
       <axis xyz="0 0 1" />
       <limit effort="100" velocity="100" />
@@ -51,7 +51,7 @@
     </transmission>
   </xacro:macro>
-  <xacro:macro name="simple_wheel" params="suffix width radius y_shift z_shift">
+  <xacro:macro name="simple_wheel" params="suffix width radius x_shift z_shift">
     <xacro:wheel  suffix="${suffix}" width="${width}" radius="${radius}"
-       x_shift="0" y_shift="${y_shift}"  z_shift="${z_shift}"/>
+       x_shift="${x_shift}" y_shift="0"  z_shift="${z_shift}"/>
   </xacro:macro>
 </robot>
